File: pcb/espairqual.kicad_pcb (KiCad board)
At the start: 4 copper layers, 56.6 x 57.7 mm, 47 parts, among them J1 24VAC, J2 PMSX003, J3 eflashy32, J4 USBC, J5 GCJA5, J7 AUX, SW1 RESET, U1 BD9G101G, U3 AMS1117-3.3, U4 ESP32-C3-MINI-1

Commit message: v4
Other:
- board text added: "espairqual v4.0 github.com/gcormier/espairqual"
- board text removed: "espairqual v3.0 github.com/gcormier/espairqual"
Changed lines of the file:
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@@
     (effects (font (size 1 1) (thickness 0.15)) (justify left bottom mirror))
   )
-  (gr_text "espairqual\nv3.0\ngithub.com/gcormier/espairqual" (at 140.543525 65.02016 90) (layer "F.SilkS")
+  (gr_text "espairqual\nv4.0\ngithub.com/gcormier/espairqual" (at 140.543525 65.02016 90) (layer "F.SilkS")
     (effects (font (size 1.5 1.5) (thickness 0.3)))
   )
