File: pcb/espairqual.kicad_pcb (KiCad board)
At the start: 4 copper layers, 56.6 x 57.7 mm, 47 parts, among them J1 24VAC, J2 PMSX003, J3 eflashy32, J4 USBC, J5 GCJA5, J7 AUX, SW1 RESET, U1 BD9G101G, U3 AMS1117-3.3, U4 ESP32-C3-MINI-1

Commit message: some tweaks
Parts:
- J1: footprint TerminalBlock_Phoenix:TerminalBlock_Phoenix_MKDS-1,5-2-5.08_1x02_P5.08mm_Horizontal -> Connector_Phoenix_MC:PhoenixContact_MC_1,5_2-G-3.81_1x02_P3.81mm_Horizontal
- moved R11 4.64 mm to (134.7, 45.0)
- moved C11 2.29 mm to (113.1, 45.3), turned to 0 degrees
- moved J4 1.68 mm to (142.1, 39.8)
- moved U4 0.30 mm to (123.4, 45.0)
- moved J1 0.13 mm to (110.3, 41.3)
Routing:
- net Net-(J4-CC2): track 7.03 -> 11.9 mm, vias 0 -> 2
- net D-: track 23.5 -> 21.5 mm
- net D+: track 26.4 -> 24.5 mm
- net Net-(J4-CC1): track 3.99 -> 5.67 mm
- net Net-(J1-Pin_2): track 7.65 -> 8.89 mm
- net /PWR5V: track 58.7 -> 59.4 mm
Other:
- outline, holes or cut-outs redrawn
- board text added: "<<hash>>"
- board text added: "espairqual v5 github.com/gcormier/espairqual"
- board text removed: "espairqual v4.0 github.com/gcormier/espairqual"

Commit message: final tweaks
Parts:
- moved F1 0.45 mm to (98.1, 43.3)
Routing:
- net /GPIO7: track 47.5 -> 46.8 mm
- net /GPIO10: track 55.2 -> 54.4 mm
- net GND: vias 56 -> 60
Other:
- outline, holes or cut-outs redrawn
- board text added: "Enclosure: Hammond 1593KBK"
- board text added: "JST-GH 1.25mm"
- board text added: "Molex Picoblade 1.25mm"
- board text removed: "Hammond 1593KBK"
