File: pcb/espairqual.kicad_sch (KiCad schematic)
At the start: 47 parts, among them J1 24VAC, J2 PMSX003, J3 eflashy32, J4 USBC, J5 GCJA5, J7 AUX, SW1 RESET, U1 BD9G101G, U3 AMS1117-3.3, U4 ESP32-C3-MINI-1

Commit message: some tweaks
Parts:
- J1: footprint TerminalBlock_Phoenix:TerminalBlock_Phoenix_MKDS-1,5-2-5.08_1x02_P5.08mm_Horizontal -> Connector_Phoenix_MC:PhoenixContact_MC_1,5_2-G-3.81_1x02_P3.81mm_Horizontal; LCSC DNP -> C480537; Part 1935161 -> (none)
Changed lines of the file:
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@@
       (effects (font (size 1.27 1.27)) (justify left))
     )
-    (property "Footprint" "TerminalBlock_Phoenix:TerminalBlock_Phoenix_MKDS-1,5-2-5.08_1x02_P5.08mm_Horizontal" (at 28.575 27.94 0)
+    (property "Footprint" "Connector_Phoenix_MC:PhoenixContact_MC_1,5_2-G-3.81_1x02_P3.81mm_Horizontal" (at 28.575 27.94 0)
       (effects (font (size 1.27 1.27)) hide)
     )
@@
       (effects (font (size 1.27 1.27)) hide)
     )
-    (property "Part" "1935161" (at 28.575 27.94 0)
+    (property "LCSC" "C480537" (at 28.575 27.94 0)
       (effects (font (size 1.27 1.27)) hide)
     )
-    (property "LCSC" "DNP" (at 28.575 27.94 0)
-      (effects (font (size 1.27 1.27)) hide)
-    )

Commit message: final tweaks
Other:
- note added: "MCU"
- note removed: "Terminal Blocks - 5mm pitch, Phoenix 1935161 / 1935174 or Chinesium equivalent"
- moved on the sheet: C1, J2, J5, R5, SW1, U4
